File: periph/station_meteo/PCB/JeeNode.sch (KiCad schematic (older format))
At the start: 32 parts, among them P1 PORT1, P2 PORT2, P3 PORT3, P4 PORT4, P5 CONN_3X2, P6 CONN_2, P7 TST, P8 TST, Q1 BSS84, Q2 BSS84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

Commit message: - Ajout info sur schéma électronique pour le brochage de la BPW34 (.sch et .pdf)
Other:
- note added: "BPW34"
Changed lines of the file:
@@
 Sheet 1 1
 Title "JeeNode shield - Sensors & GPIO"
-Date "1 nov 2013"
+Date "3 sep 2014"
 Rev "V1"
 Comp "Minbiocabanon"
@@
 	1    0    0    -1
 $EndComp
+Wire Notes Line
+	9650 3150 9650 2900
+Wire Notes Line
+	9650 2900 10150 2900
+Wire Notes Line
+	10150 2900 10150 3150
+Wire Notes Line
+	9800 2800 9800 3000
+Wire Notes Line
+	9800 2800 9950 2900
+Wire Notes Line
+	9950 2900 9800 3000
+Wire Notes Line
+	9950 2800 9950 3000
+Text Notes 9750 2700 0    60   ~ 0
+BPW34
 $EndSCHEMATC
